File: VCF1_rev1/KiCad/VCF1-mux-rev1.sch (KiCad schematic (older format))
At the start: 14 parts, among them U1 Opamp_Dual_Generic, U3 Opamp_Dual_Generic, U4 74HC4053, U5 74HC4053

Commit message: Added some initial resonance control and some other stuff.
Parts:
- removed C13, C14, C15, C16: 100nF, symbol Device:C
- removed U1, U3: Opamp_Dual_Generic, symbol Device:Opamp_Dual_Generic
- added C19: 100nF, symbol Device:C
- added C20: C, symbol Device:C
- added U6: 74HC4053, symbol 4xxx:4053
- renumbered C9 to C15, C10 to C16, C11 to C17, C12 to C18, R18 to R26, R19 to R27
Connections:
- net +5V: now also C20.1, U6.16 (VDD)
- net -5V: now also C19.1, U6.7 (VEE)
- net GND: now also C19.2, C20.2, U6.8 (VSS)
