File: VCF1_rev1/KiCad/CVpanel.kicad_sch (KiCad schematic)
At the start: 27 parts, among them J1 Thonk, J6 Thonk, SW1 SW_SPDT, SW2 SW_SPDT, SW3 SW_SPDT, SW4 SW_SPDT

Commit message: Started to populate the PCB and done some small fixes in the schematics.
Parts:
- renumbered J6 to J2
Changed lines of the file:
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@@
-(kicad_sch (version 20210621) (generator eeschema)
+(kicad_sch (version 20211123) (generator eeschema)
   (paper "A4")
-  (junction (at 121.92 69.85) (diameter 0) (color 0 0 0 0))
-  (junction (at 76.2 96.52) (diameter 0) (color 0 0 0 0))
-  (junction (at 121.92 55.88) (diameter 0) (color 0 0 0 0))
-  (junction (at 124.46 60.96) (diameter 0) (color 0 0 0 0))
-  (junction (at 222.25 96.52) (diameter 0) (color 0 0 0 0))
-  (junction (at 121.92 83.82) (diameter 0) (color 0 0 0 0))
-  (junction (at 189.23 106.68) (diameter 0) (color 0 0 0 0))
-  (junction (at 205.74 106.68) (diameter 0) (color 0 0 0 0))
-  (junction (at 30.48 58.42) (diameter 0) (color 0 0 0 0))
-  (junction (at 63.5 58.42) (diameter 0) (color 0 0 0 0))
-  (junction (at 124.46 88.9) (diameter 0) (color 0 0 0 0))
-  (junction (at 43.18 106.68) (diameter 0) (color 0 0 0 0))
-  (junction (at 46.99 44.45) (diameter 0) (color 0 0 0 0))
-  (junction (at 124.46 81.28) (diameter 0) (color 0 0 0 0))
-  (junction (at 30.48 86.36) (diameter 0) (color 0 0 0 0))
-  (junction (at 189.23 96.52) (diameter 0) (color 0 0 0 0))
-  (junction (at 96.52 86.36) (diameter 0) (color 0 0 0 0))
-  (junction (at 222.25 106.68) (diameter 0) (color 0 0 0 0))
-  (junction (at 26.67 96.52) (diameter 0) (color 0 0 0 0))
-  (junction (at 43.18 96.52) (diameter 0) (color 0 0 0 0))
-  (junction (at 124.46 86.36) (diameter 0) (color 0 0 0 0))
-  (junction (at 80.01 72.39) (diameter 0) (color 0 0 0 0))
-  (junction (at 30.48 72.39) (diameter 0) (color 0 0 0 0))
-  (junction (at 76.2 106.68) (diameter 0) (color 0 0 0 0))
-  (junction (at 205.74 96.52) (diameter 0) (color 0 0 0 0))
-  (junction (at 26.67 106.68) (diameter 0) (color 0 0 0 0))
-  (junction (at 124.46 74.93) (diameter 0) (color 0 0 0 0))
-  (junction (at 59.69 106.68) (diameter 0) (color 0 0 0 0))
-  (junction (at 59.69 96.52) (diameter 0) (color 0 0 0 0))
+  (junction (at 80.01 72.39) (diameter 0) (color 0 0 0 0)
+  )
+  (junction (at 46.99 44.45) (diameter 0) (color 0 0 0 0)
+  )
+  (junction (at 59.69 106.68) (diameter 0) (color 0 0 0 0)
+  )
+  (junction (at 26.67 96.52) (diameter 0) (color 0 0 0 0)
+  )
+  (junction (at 124.46 81.28) (diameter 0) (color 0 0 0 0)
+  )
+  (junction (at 124.46 86.36) (diameter 0) (color 0 0 0 0)
+  )
+  (junction (at 43.18 106.68) (diameter 0) (color 0 0 0 0)
+  )
+  (junction (at 189.23 96.52) (diameter 0) (color 0 0 0 0)
+  )
+  (junction (at 121.92 55.88) (diameter 0) (color 0 0 0 0)
+  )
+  (junction (at 189.23 106.68) (diameter 0) (color 0 0 0 0)
+  )
+  (junction (at 30.48 58.42) (diameter 0) (color 0 0 0 0)
+  )
+  (junction (at 26.67 106.68) (diameter 0) (color 0 0 0 0)
+  )
+  (junction (at 124.46 88.9) (diameter 0) (color 0 0 0 0)
+  )
+  (junction (at 76.2 106.68) (diameter 0) (color 0 0 0 0)
+  )
+  (junction (at 222.25 106.68) (diameter 0) (color 0 0 0 0)
+  )
+  (junction (at 205.74 96.52) (diameter 0) (color 0 0 0 0)
+  )
+  (junction (at 121.92 83.82) (diameter 0) (color 0 0 0 0)
+  )
+  (junction (at 59.69 96.52) (diameter 0) (color 0 0 0 0)
+  )
+  (junction (at 222.25 96.52) (diameter 0) (color 0 0 0 0)
+  )
+  (junction (at 43.18 96.52) (diameter 0) (color 0 0 0 0)
+  )
+  (junction (at 124.46 74.93) (diameter 0) (color 0 0 0 0)
+  )
+  (junction (at 124.46 60.96) (diameter 0) (color 0 0 0 0)
+  )
+  (junction (at 76.2 96.52) (diameter 0) (color 0 0 0 0)
+  )
+  (junction (at 96.52 86.36) (diameter 0) (color 0 0 0 0)
+  )
+  (junction (at 30.48 72.39) (diameter 0) (color 0 0 0 0)
+  )
+  (junction (at 205.74 106.68) (diameter 0) (color 0 0 0 0)
+  )
+  (junction (at 63.5 58.42) (diameter 0) (color 0 0 0 0)
+  )
+  (junction (at 121.92 69.85) (diameter 0) (color 0 0 0 0)
+  )
+  (junction (at 30.48 86.36) (diameter 0) (color 0 0 0 0)
+  )
   (wire (pts (xy 59.69 105.41) (xy 59.69 106.68))
     (stroke (width 0) (type default) (color 0 0 0 0))
@@
   (symbol (lib_id "Connector:AudioJack2_SwitchT") (at 133.35 147.32 180) (unit 1)
     (in_bom yes) (on_board yes) (fields_autoplaced)
-    (property "Reference" "J6" (id 0) (at 138.43 145.4149 0)
+    (property "Reference" "J2" (id 0) (at 138.43 145.4149 0)
       (effects (font (size 1.27 1.27)) (justify right))
     )
