File: VCF1_rev1/KiCad/MUX.kicad_sch (KiCad schematic)
At the start: 31 parts

Commit message: Lot of work on panel etc.
Parts:
- gave numbers to parts that had none: 25

Commit message: Cleaned up the first page with the overview and tried to make it a bit more readable.
Parts:
- renumbered R36 to R46, R37 to R47, R38 to R48, R39 to R49, R40 to R50, R41 to R51, R42 to R52, R43 to R53, R44 to R54, R45 to R55, R46 to R56, R47 to R57, R48 to R58, R49 to R59, R50 to R60, R51 to R61, R52 to R62, R53 to R63, R54 to R64, R55 to R65

Commit message: Drew a better symbol for LM13700 because the other one was ugly.
Parts:
- removed U5: LM13700, symbol Amplifier_Operational:LM13700
- added U20: LM13700, symbol Modular_Mayhem:LM13700
- R46, R47, R48, R49, R50, R51, R52, R53, R54, R55, R56, R57, R58, R59, R60, R61, R62, R63, R64, R65: footprint (none) -> Resistor_SMD:R_0603_1608Metric
Connections:
- net GND: now also U20.7
- net Mixer_out: now also U20.10, U20.12, U20.5
- net at R59.2, R62.2: now also U20.16
- net at R49.1: now also U20.4 (-)
- net at C8.1, R65.1: now also U20.9
- net at R53.2: now also U20.2 (DIODE_BIAS)
- net at R61.2, R63.2: now also U20.1
- net at R47.2, R55.1: now also U20.3 (+)
- net at R48.1: now also U20.13 (-)
- net at R46.2, R54.1: now also U20.14 (+)
- net at R51.2: now also U20.15 (DIODE_BIAS)
- no-connect marks 1 -> 0

Commit message: Cleanups, better names for the sheets etc.
Connections:
- no-connect marks 0 -> 1
Changed lines of the file:
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@@
 (kicad_sch (version 20210621) (generator eeschema)
   (paper "A4")
-  (junction (at 124.46 110.4901) (diameter 0) (color 0 0 0 0))
+  (junction (at 124.46 36.8301) (diameter 0) (color 0 0 0 0))
+  (junction (at 127 49.5301) (diameter 0) (color 0 0 0 0))
+  (junction (at 143.51 68.5801) (diameter 0) (color 0 0 0 0))
+  (junction (at 120.65 166.3701) (diameter 0) (color 0 0 0 0))
+  (junction (at 143.51 142.2401) (diameter 0) (color 0 0 0 0))
+  (junction (at 81.28 132.08) (diameter 0) (color 0 0 0 0))
+  (junction (at 173.99 83.82) (diameter 0) (color 0 0 0 0))
+  (junction (at 143.51 49.5301) (diameter 0) (color 0 0 0 0))
+  (junction (at 125.73 157.4801) (diameter 0) (color 0 0 0 0))
   (junction (at 149.86 81.28) (diameter 0) (color 0 0 0 0))
-  (junction (at 125.73 83.8201) (diameter 0) (color 0 0 0 0))
-  (junction (at 99.06 148.59) (diameter 0) (color 0 0 0 0))
+  (junction (at 143.51 123.19) (diameter 0) (color 0 0 0 0))
+  (junction (at 149.86 154.94) (diameter 0) (color 0 0 0 0))
   (junction (at 143.51 123.1901) (diameter 0) (color 0 0 0 0))
   (junction (at 120.65 92.7101) (diameter 0) (color 0 0 0 0))
-  (junction (at 143.51 68.5801) (diameter 0) (color 0 0 0 0))
-  (junction (at 125.73 157.4801) (diameter 0) (color 0 0 0 0))
-  (junction (at 127 49.5301) (diameter 0) (color 0 0 0 0))
-  (junction (at 143.51 123.19) (diameter 0) (color 0 0 0 0))
   (junction (at 127 123.1901) (diameter 0) (color 0 0 0 0))
+  (junction (at 99.06 148.59) (diameter 0) (color 0 0 0 0))
   (junction (at 83.82 146.05) (diameter 0) (color 0 0 0 0))
-  (junction (at 173.99 83.82) (diameter 0) (color 0 0 0 0))
-  (junction (at 149.86 154.94) (diameter 0) (color 0 0 0 0))
-  (junction (at 143.51 49.5301) (diameter 0) (color 0 0 0 0))
-  (junction (at 120.65 166.3701) (diameter 0) (color 0 0 0 0))
-  (junction (at 81.28 132.08) (diameter 0) (color 0 0 0 0))
-  (junction (at 143.51 142.2401) (diameter 0) (color 0 0 0 0))
-  (junction (at 124.46 36.8301) (diameter 0) (color 0 0 0 0))
+  (junction (at 125.73 83.8201) (diameter 0) (color 0 0 0 0))
+  (junction (at 124.46 110.4901) (diameter 0) (color 0 0 0 0))
+  (no_connect (at 38.1 182.88))
   (wire (pts (xy 186.69 81.28) (xy 184.15 81.28))
     (stroke (width 0) (type default) (color 0 0 0 0))
@@
     (stroke (width 0) (type default) (color 0 0 0 0))
   )
+  (wire (pts (xy 78.74 148.59) (xy 99.06 148.59))
+    (stroke (width 0) (type default) (color 0 0 0 0))
+  )
+  (wire (pts (xy 99.06 148.59) (xy 99.06 146.05))
+    (stroke (width 0) (type default) (color 0 0 0 0))
+  )
+  (wire (pts (xy 99.06 146.05) (xy 96.52 146.05))
+    (stroke (width 0) (type default) (color 0 0 0 0))
+  )
   (wire (pts (xy 99.06 148.59) (xy 99.06 160.02))
     (stroke (width 0) (type default) (color 0 0 0 0))
   )
-  (wire (pts (xy 99.06 148.59) (xy 99.06 146.05))
-    (stroke (width 0) (type default) (color 0 0 0 0))
-  )
-  (wire (pts (xy 99.06 146.05) (xy 96.52 146.05))
-    (stroke (width 0) (type default) (color 0 0 0 0))
-  )
-  (wire (pts (xy 78.74 148.59) (xy 99.06 148.59))
-    (stroke (width 0) (type default) (color 0 0 0 0))
-  )
   (wire (pts (xy 124.46 68.5801) (xy 124.46 36.8301))
     (stroke (width 0) (type default) (color 0 0 0 0))
@@
     (stroke (width 0) (type default) (color 0 0 0 0))
   )
+  (wire (pts (xy 143.51 142.2401) (xy 143.51 151.13))
+    (stroke (width 0) (type default) (color 0 0 0 0))
+  )
   (wire (pts (xy 143.51 132.08) (xy 143.51 142.2401))
     (stroke (width 0) (type default) (color 0 0 0 0))
   )
-  (wire (pts (xy 143.51 142.2401) (xy 143.51 151.13))
-    (stroke (width 0) (type default) (color 0 0 0 0))
-  )
   (wire (pts (xy 172.72 83.82) (xy 173.99 83.82))
     (stroke (width 0) (type default) (color 0 0 0 0))
@@
     (stroke (width 0) (type default) (color 0 0 0 0))
   )
+  (wire (pts (xy 81.28 160.02) (xy 86.36 160.02))
+    (stroke (width 0) (type default) (color 0 0 0 0))
+  )
   (wire (pts (xy 81.28 132.08) (xy 81.28 160.02))
     (stroke (width 0) (type default) (color 0 0 0 0))
   )
-  (wire (pts (xy 81.28 160.02) (xy 86.36 160.02))
-    (stroke (width 0) (type default) (color 0 0 0 0))
-  )
   (wire (pts (xy 115.57 78.7401) (xy 129.54 78.74))
     (stroke (width 0) (type default) (color 0 0 0 0))
@@
     (stroke (width 0) (type default) (color 0 0 0 0))
   )
+  (wire (pts (xy 127 49.5301) (xy 127 50.8))
+    (stroke (width 0) (type default) (color 0 0 0 0))
+  )
   (wire (pts (xy 127 41.91) (xy 127 49.5301))
     (stroke (width 0) (type default) (color 0 0 0 0))
   )
-  (wire (pts (xy 127 49.5301) (xy 127 50.8))
-    (stroke (width 0) (type default) (color 0 0 0 0))
-  )
   (wire (pts (xy 173.99 83.82) (xy 173.99 85.09))
     (stroke (width 0) (type default) (color 0 0 0 0))
@@
     (stroke (width 0) (type default) (color 0 0 0 0))
   )
+  (wire (pts (xy 78.74 146.05) (xy 83.82 146.05))
+    (stroke (width 0) (type default) (color 0 0 0 0))
+  )
   (wire (pts (xy 83.82 146.05) (xy 86.36 146.05))
     (stroke (width 0) (type default) (color 0 0 0 0))
   )
-  (wire (pts (xy 78.74 146.05) (xy 83.82 146.05))
-    (stroke (width 0) (type default) (color 0 0 0 0))
-  )

Commit message: Started to populate the PCB and done some small fixes in the schematics.
Parts:
- C10: renamed from C8; footprint (none) -> Capacitor_SMD:C_0603_1608Metric
- U4: renamed from U7; footprint (none) -> Package_SO:SOIC-14_3.9x8.7mm_P1.27mm
- U5: renamed from U20; footprint (none) -> Package_SO:SOIC-16_3.9x9.9mm_P1.27mm
- U6: footprint (none) -> Package_SO:SOIC-16_3.9x9.9mm_P1.27mm
- U7: renamed from U8; footprint (none) -> Package_SO:SOIC-16_3.9x9.9mm_P1.27mm
- renumbered R46 to R49, R47 to R50, R48 to R51, R49 to R52, R50 to R53, R51 to R54, R52 to R55, R53 to R56, R54 to R57, R55 to R58, R56 to R59, R57 to R60, R58 to R61, R59 to R62, R60 to R63, R61 to R64, R62 to R65, R63 to R66, R64 to R67, R65 to R68
Connections:
- net at R59.1, R61.1: now also U4.9 (-); no longer U4.2 (-)
- net at R53.2, R62.1: now also U4.10 (+); no longer U4.3 (+)
- net at R55.2, R64.1: now also U4.12 (+); no longer U4.5 (+)
- net at R60.1, R63.1: now also U4.13 (-); no longer U4.6 (-)
- net at R61.2, R65.1: now also U4.8; no longer U4.1

Commit message: Placed more components on the PCB.
Parts:
- added C10, C11: C, Capacitor_SMD:C_0603_1608Metric, symbol Device:C
- renumbered C10 to C12
Connections:
- net at R59.1, R61.1, U4.9 (-): now also C10.1
- net at R56.2, U5.2 (DIODE_BIAS): now also R55.2, R64.1, U4.12 (+)
- net at R63.2, R66.1: now also U4.14, C11.2
- net at R60.1, R63.1, U4.13 (-): now also C11.1
- net at R61.2, R65.1, U4.8: now also C10.2
Other:
- moved on the sheet: R50, R52, R53, R56, R58, R60, R63, R64, R66, R67, U4C, U5C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
