File: VCF1_rev1/KiCad/Power.kicad_sch (KiCad schematic)
At the start: 18 parts, among them J5 Conn_02x05_Odd_Even, U1 Opamp_Quad, U10 CEM3350, U14 Opamp_Quad, U16 CEM3350, U4 Opamp_Quad, U5 LM13700

Commit message: Started to populate the PCB and done some small fixes in the schematics.
Parts:
- removed U5: LM13700, symbol Modular_Mayhem:LM13700
- added C26, C27, C30, C31, C32, C35: 100nF, Capacitor_SMD:C_0603_1608Metric, symbol Device:C
- added U10: Opamp_Quad, Package_SO:SOIC-14_3.9x8.7mm_P1.27mm, symbol Device:Opamp_Quad
- added U11, U8: 74HC4053, Package_SO:SOIC-16_3.9x9.9mm_P1.27mm, symbol Modular_Mayhem:74HC4053
- C22: renamed from C18; footprint (none) -> Capacitor_SMD:C_0603_1608Metric
- C23: renamed from C19; footprint (none) -> Capacitor_SMD:C_0603_1608Metric
- C24: renamed from C20; footprint (none) -> Capacitor_SMD:C_0603_1608Metric
- C25: renamed from C21; footprint (none) -> Capacitor_SMD:C_0603_1608Metric
- C28: renamed from C22; footprint (none) -> Capacitor_SMD:C_0603_1608Metric
- C29: renamed from C23; footprint (none) -> Capacitor_SMD:C_0603_1608Metric
- C33: renamed from C24; footprint (none) -> Capacitor_SMD:C_0603_1608Metric
- C34: renamed from C25; footprint (none) -> Capacitor_SMD:C_0603_1608Metric
- C36: renamed from C26; footprint (none) -> Capacitor_SMD:C_0603_1608Metric
- C37: renamed from C27; footprint (none) -> Capacitor_SMD:C_0603_1608Metric
- U1, U4: footprint (none) -> Package_SO:SOIC-14_3.9x8.7mm_P1.27mm
- U12: renamed from U14; footprint (none) -> Package_SO:SOIC-14_3.9x8.7mm_P1.27mm
- U3: renamed from U16; footprint (none) -> Package_SO:SOIC-16_3.9x9.9mm_P1.27mm
- U9: renamed from U10; footprint (none) -> Package_SO:SOIC-16_3.9x9.9mm_P1.27mm
- renumbered J5 to J6
Connections:
- net +10V: now also C26.1, C30.1, C32.2, U10.4 (V+), U11.16 (Vcc), U8.16 (Vcc)
- net -10V: now also C27.2, C31.1, C35.2, U10.11 (V-), U11.7 (Vee), U8.7 (Vee)
- net GND: now also C26.2, C27.1, C30.2, C31.2, C32.1, C35.1, U11.6 (~{E}), U11.8 (GND), U8.6 (~{E}), U8.8 (GND)

Commit message: Placed more components on the PCB.
Parts:
- renumbered C22 to C30, C23 to C31, C24 to C32, C25 to C33, C26 to C34, C27 to C35, C28 to C36, C29 to C37, C30 to C38, C31 to C39, C32 to C40, C33 to C41, C34 to C42, C35 to C43, C36 to C44, C37 to C45
Changed lines of the file:
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@@
   (symbol (lib_id "Device:C") (at 248.92 90.17 0) (mirror y) (unit 1)
     (in_bom yes) (on_board yes) (fields_autoplaced)
-    (property "Reference" "C37" (id 0) (at 245.11 88.8999 0)
+    (property "Reference" "C45" (id 0) (at 245.11 88.8999 0)
       (effects (font (size 1.27 1.27)) (justify left))
     )
@@
   (symbol (lib_id "Device:C") (at 248.92 80.01 0) (mirror y) (unit 1)
     (in_bom yes) (on_board yes) (fields_autoplaced)
-    (property "Reference" "C36" (id 0) (at 245.11 78.7399 0)
+    (property "Reference" "C44" (id 0) (at 245.11 78.7399 0)
       (effects (font (size 1.27 1.27)) (justify left))
     )
@@
   (symbol (lib_id "Device:C") (at 67.31 156.21 0) (unit 1)
     (in_bom yes) (on_board yes) (fields_autoplaced)
-    (property "Reference" "C23" (id 0) (at 71.12 154.9399 0)
+    (property "Reference" "C31" (id 0) (at 71.12 154.9399 0)
       (effects (font (size 1.27 1.27)) (justify left))
     )
@@
   (symbol (lib_id "Device:C") (at 217.17 134.62 0) (unit 1)
     (in_bom yes) (on_board yes) (fields_autoplaced)
-    (property "Reference" "C33" (id 0) (at 220.98 133.3499 0)
+    (property "Reference" "C41" (id 0) (at 220.98 133.3499 0)
       (effects (font (size 1.27 1.27)) (justify left))
     )
@@
   (symbol (lib_id "Device:C") (at 69.85 73.66 0) (unit 1)
     (in_bom yes) (on_board yes) (fields_autoplaced)
-    (property "Reference" "C25" (id 0) (at 73.66 72.3899 0)
+    (property "Reference" "C33" (id 0) (at 73.66 72.3899 0)
       (effects (font (size 1.27 1.27)) (justify left))
     )
@@
   (symbol (lib_id "Device:C") (at 114.3 71.12 0) (unit 1)
     (in_bom yes) (on_board yes) (fields_autoplaced)
-    (property "Reference" "C27" (id 0) (at 118.11 69.8499 0)
+    (property "Reference" "C35" (id 0) (at 118.11 69.8499 0)
       (effects (font (size 1.27 1.27)) (justify left))
     )
@@
   (symbol (lib_id "Device:C") (at 114.3 60.96 0) (unit 1)
     (in_bom yes) (on_board yes) (fields_autoplaced)
-    (property "Reference" "C26" (id 0) (at 118.11 59.6899 0)
+    (property "Reference" "C34" (id 0) (at 118.11 59.6899 0)
       (effects (font (size 1.27 1.27)) (justify left))
     )
@@
   (symbol (lib_id "Device:C") (at 137.16 133.35 0) (unit 1)
     (in_bom yes) (on_board yes) (fields_autoplaced)
-    (property "Reference" "C29" (id 0) (at 140.97 132.0799 0)
+    (property "Reference" "C37" (id 0) (at 140.97 132.0799 0)
       (effects (font (size 1.27 1.27)) (justify left))
     )
@@
   (symbol (lib_id "Device:C") (at 204.47 46.99 180) (unit 1)
     (in_bom yes) (on_board yes) (fields_autoplaced)
-    (property "Reference" "C32" (id 0) (at 208.28 45.7199 0)
+    (property "Reference" "C40" (id 0) (at 208.28 45.7199 0)
       (effects (font (size 1.27 1.27)) (justify right))
     )
@@
   (symbol (lib_id "Device:C") (at 137.16 123.19 0) (unit 1)
     (in_bom yes) (on_board yes) (fields_autoplaced)
-    (property "Reference" "C28" (id 0) (at 140.97 121.9199 0)
+    (property "Reference" "C36" (id 0) (at 140.97 121.9199 0)
       (effects (font (size 1.27 1.27)) (justify left))
     )
@@
   (symbol (lib_id "Device:C") (at 161.29 54.61 0) (unit 1)
     (in_bom yes) (on_board yes) (fields_autoplaced)
-    (property "Reference" "C30" (id 0) (at 165.1 53.3399 0)
+    (property "Reference" "C38" (id 0) (at 165.1 53.3399 0)
       (effects (font (size 1.27 1.27)) (justify left))
     )
@@
   (symbol (lib_id "Device:C") (at 175.26 77.47 0) (unit 1)
     (in_bom yes) (on_board yes) (fields_autoplaced)
-    (property "Reference" "C31" (id 0) (at 179.07 76.1999 0)
+    (property "Reference" "C39" (id 0) (at 179.07 76.1999 0)
       (effects (font (size 1.27 1.27)) (justify left))
     )
@@
   (symbol (lib_id "Device:C") (at 218.44 69.85 180) (unit 1)
     (in_bom yes) (on_board yes) (fields_autoplaced)
-    (property "Reference" "C35" (id 0) (at 222.25 68.5799 0)
+    (property "Reference" "C43" (id 0) (at 222.25 68.5799 0)
       (effects (font (size 1.27 1.27)) (justify right))
     )
@@
   (symbol (lib_id "Device:C") (at 67.31 146.05 0) (unit 1)
     (in_bom yes) (on_board yes) (fields_autoplaced)
-    (property "Reference" "C22" (id 0) (at 71.12 144.7799 0)
+    (property "Reference" "C30" (id 0) (at 71.12 144.7799 0)
       (effects (font (size 1.27 1.27)) (justify left))
     )
@@
   (symbol (lib_id "Device:C") (at 69.85 63.5 0) (unit 1)
     (in_bom yes) (on_board yes) (fields_autoplaced)
-    (property "Reference" "C24" (id 0) (at 73.66 62.2299 0)
+    (property "Reference" "C32" (id 0) (at 73.66 62.2299 0)
       (effects (font (size 1.27 1.27)) (justify left))
     )
@@
   (symbol (lib_id "Device:C") (at 217.17 144.78 0) (unit 1)
     (in_bom yes) (on_board yes) (fields_autoplaced)
-    (property "Reference" "C34" (id 0) (at 220.98 143.5099 0)
-      (effects (font (size 1.27 1.27)) (justify left))
-    )
+    (property "Reference" "C42" (id 0) (at 220.98 143.5099 0)
+      (effects (font (size 1.27 1.27)) (justify left))
+    )
