File: VCF1_rev1/KiCad/VCF1_rev1.kicad_sch (KiCad schematic)
At the start: 0 parts

Commit message: Cleanups, better names for the sheets etc.
Other:
- removed sheet Input_mixer
- added sheet CVpanel (CVpanel.kicad_sch)
- sheet Audiopanel ports: added Audio_out; removed Frequency_sum_VCF1, Frequency_sum_VCF2, Frequency_sum_VCF3, Frequency_sum_VCF4, Resonance_sum_VCF1, Resonance_sum_VCF2, Resonance_sum_VCF3, Resonance_sum_VCF4, VCA1_CV, VCA2_CV, VCA3_CV
